File: buck100.kicad_pcb (KiCad board)
At the start: 2 copper layers, 10.5 x 19.5 mm, 15 parts, among them J1 Conn_01x03_Male, U2 LM5163DDAR

Commit message: docs, vias
Parts:
- C1: value ~ -> 2200 pF, 100 V
- C6: value ~ -> 56pF, 50V; footprint Capacitor_SMD:C_0805_2012Metric_Pad1.18x1.45mm_HandSolder -> Capacitor_SMD:C_0603_1608Metric_Pad1.08x0.95mm_HandSolder
- C7: value 2200 pF, 50 V, X7R, 10% -> 2200 pF, 50 V
Routing:
- net VIN: track 9.31 -> 8.74 mm
- net SW: vias 3 -> 4
- net GND: vias 1 -> 3

Commit message: minor changes
Parts:
- removed R3: 33k, Resistor_SMD:R_0805_2012Metric
- R5: value 33k -> 100k
- moved R1 0.64 mm to (147.3, 99.5)
- moved R2 0.64 mm to (147.3, 103.0)
Routing:
- net FB: track 10.5 -> 8.52 mm
- net +3.3V: track 24.8 -> 22.8 mm
- net GND: track 9.91 -> 9.28 mm
Other:
- board text added: "Ra"
- board text added: "Rfb1"
- board text added: "Rfb2"
- board text added: "Rt"
