File: buck100.kicad_sch (KiCad schematic)
At the start: 17 parts, among them J1 Conn_01x03_Male, U2 LM5163DDAR

Commit message: docs, vias
Parts:
- C1: value (none) -> 2200 pF, 100 V
- C6: value (none) -> 56pF, 50V; footprint Capacitor_SMD:C_0805_2012Metric_Pad1.18x1.45mm_HandSolder -> Capacitor_SMD:C_0603_1608Metric_Pad1.08x0.95mm_HandSolder; Digikey (none) -> 0603N560J500CT; Ref GCM155R71H222KA37D -> (none)
- C7: value 2200 pF, 50 V, X7R, 10% -> 2200 pF, 50 V
- R3: now not fitted; now left out of the parts list
- R4: value (none) -> ~
- R5: value 33k -> 100k
Other:
- note added: "LM5163 100Vmax 0.5A LM5164 100Vmax 1.0A LM5168 120Vmax 0.3A LM5169 120Vmax 0.65A"
- note added: "TI Design Tool"
- moved on the sheet: C1, C2, C6, L1, R1, R2, R4

Commit message: minor changes
Other:
- note added: "Rfb1"
- note added: "Rfb2"
Changed lines of the file:
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@@
+	(wire
+		(pts
+			(xy 135.89 59.69) (xy 146.05 59.69)
+		)
+		(stroke
+			(width 0)
+			(type default)
+		)
+	)
 	(wire
 		(pts
@@
 	(wire
 		(pts
-			(xy 135.89 59.69) (xy 146.05 59.69)
-		)
-		(stroke
-			(width 0)
-			(type default)
-		)
-	)
-	(wire
-		(pts
 			(xy 185.42 59.69) (xy 185.42 72.39)
 		)
@@
 			(width 0)
 			(type default)
+		)
+	)
+	(text "Rfb1\n"
+		(exclude_from_sim no)
+		(at 180.594 74.93 0)
+		(effects
+			(font
+				(size 1.27 1.27)
+			)
 		)
 	)
@@
 			)
 			(href "https://www.ti.com/tool/LM5163-LM5164DESIGN-CALC#downloads")
+		)
+	)
+	(text "Rfb2\n"
+		(exclude_from_sim no)
+		(at 179.832 90.424 0)
+		(effects
+			(font
+				(size 1.27 1.27)
+			)
 		)
 	)
@@
 	(global_label "SW"
 		(shape input)
-		(at 146.05 59.69 90)
+		(at 135.89 59.69 180)
 		(fields_autoplaced yes)
 		(effects
@@
 				(size 1.27 1.27)
 			)
-			(justify left)
+			(justify right)
 		)
 		(property "Intersheetrefs" "${INTERSHEET_REFS}"
-			(at 146.05 54.0439 90)
-			(effects
-				(font
-					(size 1.27 1.27)
-				)
-				(justify left)
+			(at 130.2439 59.69 0)
+			(effects
+				(font
+					(size 1.27 1.27)
+				)
+				(justify right)
 				(hide yes)
 			)
@@
 		(exclude_from_sim yes)
 		(in_bom no)
-		(on_board yes)
+		(on_board no)
 		(dnp yes)
 		(fields_autoplaced yes)
