File: buck100.kicad_sch (KiCad schematic)
At the start: 17 parts, among them J1 Conn_01x03_Male, U2 LM5163DDAR

Commit message: doc
Parts:
- C7: value 2200 pF, 50 V -> 2200 pF, 50 V, X74
Changed lines of the file:
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@@
 			)
 		)
-		(property "Value" "2200 pF, 50 V"
+		(property "Value" "2200 pF, 50 V, X74"
 			(at 118.11 69.596 0)
 			(effects
@@
 			)
 		)
-		(property "Description" "Unpolarized capacitor, small symbol"
+		(property "Description" "Unpolarized capacitor, small symbol can also be 50V"
 			(at 125.73 76.2 0)
 			(effects
@@
 		)
 		(property "Value" "100k"
-			(at 95.25 91.44 0)
-			(effects
-				(font
+			(at 92.075 93.345 0)
+			(effects
+				(font
